File: kicad/Triton.kicad_sch (KiCad schematic)
At the start: 0 parts

Commit message: split schematic into separate sheets. Started populating CPU sheet.
Other:
- added sheet CPU (cpu.kicad_sch)
- added sheet KBD Port (kbd.kicad_sch)
- added sheet Memory (memory.kicad_sch)
- added sheet PSU (psu.kicad_sch)
- added sheet Tape IO (tape.kicad_sch)
- added sheet VDU (vdu.kicad_sch)
- title: (none) -> Triton 8080 One-Board Home Computer
